File: Hardware/C-Audio Input Board/3,5mm.kicad_sch (KiCad schematic)
At the start: 8 parts, among them J33 3.5mm, J34 +, J35 -, J36 GND, J37 +_sw, J38 -_sw, J39 Conn_01x05_Socket, J40 Conn_01x03_Socket

Commit message: added mouser and reichelt numbers to BOM
Parts:
- J33: Reichelt Link (none) -> https://www.reichelt.de/de/de/shop/produkt/klinkeneinbaubuc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; Reichelt Nr. (none) -> EBS 35
- J39: Reichelt Nr. (none) -> JST EH5P ST
- J40: Reichelt Nr. (none) -> JST EH3P ST
Changed lines of the file:
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@@
+			)
+		)
+		(property "Reichelt Nr." "JST EH5P ST"
+			(at 116.205 69.85 0)
+			(effects
+				(font
+					(size 1.27 1.27)
+				)
 			)
 		)
@@
 			)
 		)
+		(property "Mouser Nr." ""
+			(at 74.93 72.39 0)
+			(effects
+				(font
+					(size 1.27 1.27)
+				)
+				(hide yes)
+			)
+		)
+		(property "Mouser Link" ""
+			(at 74.93 72.39 0)
+			(effects
+				(font
+					(size 1.27 1.27)
+				)
+				(hide yes)
+			)
+		)
+		(property "Reichelt Nr." "EBS 35"
+			(at 74.93 72.39 0)
+			(effects
+				(font
+					(size 1.27 1.27)
+				)
+				(hide yes)
+			)
+		)
+		(property "Reichelt Link" "https://www.reichelt.de/de/de/shop/produkt/klinkeneinbaubuchse_3_5_mm_stereo-7301"
+			(at 74.93 72.39 0)
+			(effects
+				(font
+					(size 1.27 1.27)
+				)
+				(hide yes)
+			)
+		)
 		(pin "S"
 		)
@@
 			)
 		)
+		(property "Reichelt Nr." " JST EH3P ST"
+			(at 116.205 82.55 0)
+			(effects
+				(font
+					(size 1.27 1.27)
+				)
+			)
+		)
